File: spudpole/modctl/hardware/1.0/kicad/modctl-v1.0.kicad_pcb (KiCad board)
At the start: 2 copper layers, 75 x 75 mm, 42 parts, among them J1 SWITCH INPUTS, J2 RELAY OUTPUTS, J3 M12-5PIN, SW1 PRGW0, SW2 PRGW1, SW3 INSTANCE, U1 POWER, U2 W0UP, U3 CNY74-4H, U4 W0DN, U5 W1UP, U6 W1DN, U7 Teensy_3.2, U8 TEC2-2411WI, U9 MCP2551-I-P

Commit message: README...
Parts:
- added JP5: SCR, Connector_PinHeader_2.54mm:PinHeader_1x02_P2.54mm_Vertical, F.Cu at (15.2, 31.8)
- J3: footprint TerminalBlock_Phoenix:TerminalBlock_Phoenix_MPT-0,5-4-2.54_1x04_P2.54mm_Horizontal -> TerminalBlock_Phoenix:TerminalBlock_Phoenix_MPT-0,5-5-2.54_1x05_P2.54mm_Horizontal
- JP1: value Jumper_2_Open -> 2-4
- JP2: value Jumper_2_Open -> 2-6
- JP3: value Jumper_2_Open -> 2-8
- JP4: value Jumper_2_Open -> 2-10
- moved J3 1.91 mm to (27.3, 22.2)
Routing:
- net Net-(J3-Pad5): track 0.00 -> 28.0 mm
- net Net-(J3-Pad2): track 28.5 -> 30.5 mm
- net Net-(J3-Pad3): track 16.8 -> 14.9 mm
- net Net-(F1-Pad1): track 24.8 -> 26.7 mm
- net Net-(J3-Pad4): track 20.8 -> 19.2 mm
Other:
- board text added: "SCR"
