File: spudpole/modint/hardware/1.0/kicad/modint-v1.0.kicad_pcb (KiCad board)
At the start: 2 copper layers, 75 x 75 mm, 43 parts, among them J1 SENSOR, J2 Screw_Terminal_01x05, J3 NMEA, J4 RELAYS, K1 RS-RELAY, K2 RS-RELAY, Q1 2N2219, Q2 2N2219, SW1 INSTANCE/TERM, U1 CNY74-4H, U2 Teensy_3.2, U3 TEC2-2411WI, U4 MCP2551-I-P

Commit message: Slight PCB tweaks
Parts:
- J3: value NMEA -> M12-5PIN
- K1, K2: value RS-RELAY -> SANYOU_SRD_Form_C
- U1: footprint Package_DIP:DIP-16_W7.62mm -> Package_DIP:DIP-16_W7.62mm_LongPads
- moved U1 0.64 mm to (176.2, 112.4)
Connections:
- K1 pad 6: (no net) -> Net-(J4-Pad2)
- K2 pad 6: (no net) -> Net-(J4-Pad5)
- U1 pad 11: GND -> Net-(U1-Pad11)
- U1 pad 12: Net-(U1-Pad12) -> GND
- U1 pad 15: GND -> Net-(U1-Pad15)
- U1 pad 16: Net-(U1-Pad16) -> GND
- U1 pad 3: Net-(D2-Pad1) -> Net-(D1-Pad2)
- U1 pad 4: Net-(D1-Pad2) -> Net-(D2-Pad1)
- U1 pad 7: Net-(D4-Pad1) -> Net-(D1-Pad2)
- U1 pad 8: Net-(D1-Pad2) -> Net-(D4-Pad1)
- U2 pad 10: Net-(U1-Pad16) -> Net-(U1-Pad15)
- U2 pad 13: Net-(U1-Pad12) -> Net-(U1-Pad11)
Routing:
- net Net-(U1-Pad11): track 0.00 -> 80.3 mm
- net Net-(U1-Pad12): track 77.1 -> 0.00 mm
- net Net-(U1-Pad15): track 0.00 -> 65.1 mm
- net Net-(U1-Pad16): track 61.6 -> 0.00 mm
- net Net-(D1-Pad2): track 133.6 -> 138.7 mm
- net Net-(D2-Pad1): track 58.5 -> 61.4 mm
- net Net-(J4-Pad5): track 26.2 -> 28.8 mm
- net Net-(J4-Pad2): track 26.2 -> 28.8 mm
- net Net-(D4-Pad1): track 64.8 -> 66.8 mm

Commit message: Slight PCB tweaks
Parts:
- removed R13: 120R, Resistor_THT:R_Axial_DIN0204_L3.6mm_D1.6mm_P5.08mm_Horizontal
- D5: footprint LED_THT:LED_Rectangular_W5.0mm_H2.0mm-3Pins -> LED_THT:LED_Rectangular_W3.0mm_H2.0mm
- R1, R2, R3, R4: value 3K3 -> 1K4
- R10, R7, R9: value 1K -> 200R
- SW1: value INSTANCE/TERM -> INSTANCE; footprint PDJR:DIP-18_297_ELL -> Button_Switch_THT:SW_DIP_SPSTx08_Slide_6.7x21.88mm_W7.62mm_P2.54mm_LowProfile
- moved R7 29.3 mm to (207.9, 125.7), turned to 180 degrees
- moved SW1 9.66 mm to (168.6, 141.6), turned to 180 degrees
- moved D5 4.02 mm to (204.1, 129.5), turned to 0 degrees
Connections:
- D5 pad 1: GND -> Net-(D5-Pad1)
- D8 pad 1: Net-(D8-Pad1) -> Net-(D5-Pad2)
- D9 pad 1: Net-(D8-Pad1) -> Net-(D5-Pad2)
- F1 pad 1: Net-(D8-Pad1) -> Net-(D5-Pad2)
- K1 pad 9: Net-(D8-Pad1) -> Net-(D5-Pad2)
- K2 pad 9: Net-(D8-Pad1) -> Net-(D5-Pad2)
- R10 pad 2: Net-(D8-Pad1) -> Net-(D5-Pad2)
- R7 pad 1: Net-(D5-Pad2) -> Net-(R7-Pad1)
- R7 pad 2: Net-(D8-Pad1) -> Net-(D5-Pad1)
- R9 pad 2: Net-(D8-Pad1) -> Net-(D5-Pad2)
- SW1 pad 10: Net-(R13-Pad2) -> Net-(SW1-Pad10)
- SW1 pad 9: Net-(J3-Pad3) -> Net-(SW1-Pad9)
- U2 pad 12: Net-(D5-Pad3) -> Net-(R7-Pad1)
- U2 pad 15: Net-(SW1-Pad18) -> Net-(SW1-Pad16)
- U2 pad 16: Net-(SW1-Pad17) -> Net-(SW1-Pad15)
- U2 pad 17: Net-(SW1-Pad16) -> Net-(SW1-Pad14)
- U2 pad 18: Net-(SW1-Pad15) -> Net-(SW1-Pad13)
- U2 pad 19: Net-(SW1-Pad14) -> Net-(SW1-Pad12)
- U2 pad 20: Net-(SW1-Pad13) -> Net-(SW1-Pad11)
- U2 pad 21: Net-(SW1-Pad12) -> Net-(SW1-Pad10)
- U2 pad 22: Net-(SW1-Pad11) -> Net-(SW1-Pad9)
- U2 pad 28: Net-(D8-Pad1) -> Net-(D5-Pad2)
- U3 pad 6: Net-(D8-Pad1) -> Net-(D5-Pad2)
- U4 pad 3: Net-(D8-Pad1) -> Net-(D5-Pad2)
Routing:
- net Net-(D8-Pad1): track 233.8 -> 0.00 mm
- net Net-(D5-Pad2): track 32.1 -> 241.5 mm
- net Net-(R7-Pad1): track 0.00 -> 120.5 mm
- net Net-(D5-Pad3): track 117.5 -> 0.00 mm
- net Net-(J3-Pad3): track 104.8 -> 31.3 mm
- net Net-(R13-Pad2): track 20.6 -> 0.00 mm
- net Net-(J3-Pad4): track 40.9 -> 27.7 mm
- net Net-(SW1-Pad9): track 0.00 -> 6.92 mm
- net Net-(SW1-Pad10): track 0.00 -> 6.92 mm
- net Net-(SW1-Pad18): track 6.68 -> 0.00 mm
- net Net-(SW1-Pad17): track 6.68 -> 0.00 mm
- net Net-(D5-Pad1): track 0.00 -> 4.34 mm
Other:
- board text removed: "T"

Commit message: Building Gerber files
Parts:
- added C3: 100nF, Capacitor_THT:CP_Radial_D5.0mm_P2.50mm, F.Cu at (155.9, 95.9)
- added C4: 100nF, Capacitor_THT:CP_Radial_D5.0mm_P2.50mm, F.Cu at (155.2, 104.8)
- added JP1: Jumper_NO_Small, Jumper:SolderJumper-3_P1.3mm_Open_Pad1.0x1.5mm, F.Cu at (187.7, 99.7)
- added R13: 4K7, Resistor_THT:R_Axial_DIN0204_L3.6mm_D1.6mm_P5.08mm_Horizontal, F.Cu at (159.7, 118.1)
- C1, C2: footprint Capacitor_THT:C_Disc_D7.5mm_W4.4mm_P5.00mm -> Capacitor_THT:CP_Radial_D5.0mm_P2.50mm
- D1, D2, D3, D4: value D_Small -> 1N4007
- J1: value SENSOR -> NPN SENSOR; footprint TerminalBlock_Phoenix:TerminalBlock_Phoenix_MPT-0,5-3-2.54_1x03_P2.54mm_Horizontal -> PDJR:TerminalBlock_Phoenix_MPT-0,5-3-2.54_1x03_P2.54mm_Horizontal
- R1, R2, R3, R4: value 1K4 -> 1K4, 1W
- R5, R6: value 1K -> 4K7
- R7: value 200R -> 200R, 125mW
- R8: value 10K -> 4K7; footprint Resistor_THT:R_Axial_DIN0204_L3.6mm_D1.6mm_P5.08mm_Horizontal -> Resistor_THT:R_Axial_DIN0204_L3.6mm_D1.6mm_P2.54mm_Vertical
- REF** (x2): value MountingHole_2.7mm_M2.5_Pad -> M2.7
- moved R8 19.8 mm to (160.3, 104.8), turned to 90 degrees
- moved R6 7.62 mm to (176.2, 120.7), turned to 180 degrees
- moved C1 7.10 mm to (171.8, 91.4)
- moved C2 5.99 mm to (171.8, 96.5)
- moved U4 5.75 mm to (160.3, 90.8)
- moved R12 5.68 mm to (180.0, 96.5), turned to 90 degrees
- moved R11 5.24 mm to (177.5, 96.5), turned to 90 degrees
- moved R5 4.58 mm to (176.2, 124.5), turned to 180 degrees
- moved F2 4.02 mm to (207.9, 90.2)
- moved F1 2.84 mm to (139.4, 153.7)
- moved J3 2.54 mm to (191.4, 94.0)
- moved D6 1.27 mm to (204.1, 137.2)
- moved D7 1.27 mm to (204.1, 144.8)
- moved J1 1.27 mm to (154.6, 154.9)
- moved J4 1.27 mm to (180.0, 154.9)
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Connections:
- U2 pad 27: (no net) -> GND
Routing:
- net Net-(J1-Pad3): track 31.0 -> 41.5 mm
- net Net-(D1-Pad2): track 138.7 -> 128.5 mm, vias 0 -> 1
- net Net-(J3-Pad4): track 27.7 -> 18.5 mm
- net Net-(R6-Pad2): track 24.3 -> 15.9 mm, vias 1 -> 0
- net Net-(J3-Pad2): track 19.7 -> 27.6 mm
- net Net-(J3-Pad3): track 31.3 -> 23.8 mm
- net Net-(C3-Pad1): track 241.5 -> 247.8 mm
- net Net-(U2-Pad6): track 37.7 -> 43.9 mm
- net Net-(U2-Pad5): track 42.7 -> 48.7 mm
- net Net-(F2-Pad1): track 12.7 -> 18.1 mm
- net Net-(Q1-Pad2): track 8.90 -> 3.81 mm
- net Net-(C2-Pad2): track 3.89 -> 8.43 mm
- net Net-(R7-Pad1): track 120.5 -> 116.8 mm, vias 0 -> 1
- net Net-(F1-Pad2): track 18.6 -> 22.2 mm
- net Net-(F2-Pad2): track 9.95 -> 13.2 mm
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Other:
- board text added: "DOWN"
- board text added: "PDJR"
- board text added: "PWR/TX"
- board text added: "modint 1.0"

Commit message: Moved GPIO definitions into defines
Other:
- board text removed: "DOWN"
- board text removed: "PDJR"
- board text removed: "PWR/TX"
- board text removed: "modint 1.0"
Changed lines of the file:
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@@
   (general
     (thickness 1.6)
-    (drawings 66)
+    (drawings 57)
     (tracks 300)
     (zones 0)
@@
   )
   (layers
-    (0 F.Cu signal)
+    (0 F.Cu signal hide)
     (31 B.Cu signal hide)
     (33 F.Adhes user hide)
@@
     (39 F.Mask user hide)
     (40 Dwgs.User user hide)
-    (41 Cmts.User user hide)
-    (42 Eco1.User user hide)
+    (41 Cmts.User user)
+    (42 Eco1.User user)
     (43 Eco2.User user hide)
     (44 Edge.Cuts user)
@@
     )
   )
+  (gr_circle (center 200 98) (end 203.81 98) (layer Eco1.User) (width 0.15))
+  (gr_line (start 196.19 97.365) (end 203.81 97.365) (layer Eco1.User) (width 0.15))
+  (gr_line (start 196.19 98.635) (end 203.81 98.635) (layer Eco1.User) (width 0.15))
+  (gr_circle (center 147 98) (end 150.81 98) (layer Eco1.User) (width 0.15))
+  (gr_line (start 143.19 97.365) (end 150.81 97.365) (layer Eco1.User) (width 0.15))
+  (gr_line (start 143.19 98.635) (end 150.81 98.635) (layer Eco1.User) (width 0.15))
+  (gr_circle (center 147 151) (end 150.81 151) (layer Eco1.User) (width 0.15))
+  (gr_line (start 143.19 150.365) (end 150.81 150.365) (layer Eco1.User) (width 0.15))
+  (gr_line (start 143.19 151.635) (end 150.81 151.635) (layer Eco1.User) (width 0.15))
+  (gr_circle (center 200 151) (end 203.81 151) (layer Eco1.User) (width 0.15))
+  (gr_line (start 196.19 150.365) (end 203.81 150.365) (layer Eco1.User) (width 0.15))
+  (gr_line (start 196.19 151.635) (end 203.81 151.635) (layer Eco1.User) (width 0.15))
   (gr_line (start 158.42 158.75) (end 160.96 158.75) (layer F.SilkS) (width 0.15))
-  (gr_text "modint 1.0" (at 138.1 114.3) (layer Cmts.User)
-    (effects (font (size 4 2) (thickness 0.5) italic) (justify left))
-  )
-  (gr_text PDJR (at 138.1 101.6) (layer Cmts.User)
-    (effects (font (size 10 6) (thickness 1.5) italic) (justify left))
-  )
-  (gr_circle (center 200 98) (end 197.46 96.73) (layer Cmts.User) (width 0.15))
-  (gr_circle (center 198.73 99.27) (end 199.06 99.06) (layer Cmts.User) (width 0.15))
-  (gr_circle (center 201.27 99.27) (end 201.6 99.06) (layer Cmts.User) (width 0.15))
-  (gr_circle (center 198.73 96.73) (end 199.06 96.52) (layer Cmts.User) (width 0.15))
-  (gr_circle (center 201.27 96.73) (end 201.6 96.52) (layer Cmts.User) (width 0.15))
-  (gr_circle (center 200 98) (end 200.33 97.79) (layer Cmts.User) (width 0.15))
-  (gr_circle (center 200 98) (end 202.87 97.79) (layer Cmts.User) (width 0.15))
-  (gr_circle (center 200 98) (end 205.41 99.06) (layer Cmts.User) (width 0.15))
-  (gr_circle (center 200 98) (end 206.68 97.79) (layer Cmts.User) (width 0.15))
-  (gr_text UP (at 201.5 144.5) (layer Cmts.User)
-    (effects (font (size 3 2) (thickness 0.3)) (justify right))
-  )
-  (gr_text DOWN (at 201.5 137) (layer Cmts.User)
-    (effects (font (size 3 2) (thickness 0.3)) (justify right))
-  )
-  (gr_text PWR/TX (at 201.5 129.5) (layer Cmts.User)
-    (effects (font (size 3 2) (thickness 0.3)) (justify right))
-  )
   (gr_line (start 123.5 161.5) (end 133.5 164.5) (layer Cmts.User) (width 0.15))
   (gr_line (start 123.5 87.5) (end 123.5 161.5) (layer Cmts.User) (width 0.15))
@@
   (gr_line (start 223.5 87.5) (end 223.5 161.5) (layer Cmts.User) (width 0.15))
   (gr_line (start 213.5 84.5) (end 223.5 87.5) (layer Cmts.User) (width 0.15))
-  (gr_circle (center 205.5 129.5) (end 207 129.5) (layer Cmts.User) (width 0.15))
-  (gr_circle (center 205.5 144.75) (end 207 144.75) (layer Cmts.User) (width 0.15))
-  (gr_circle (center 205.5 137) (end 207 137) (layer Cmts.User) (width 0.15))
-  (gr_circle (center 200 151) (end 206 151) (layer Eco1.User) (width 0.15))
-  (gr_circle (center 147 151) (end 153 151) (layer Eco1.User) (width 0.15))
-  (gr_circle (center 147 98) (end 153 98) (layer Eco1.User) (width 0.15))
-  (gr_circle (center 200 98) (end 206 98) (layer Eco1.User) (width 0.15))
   (gr_line (start 133.5 84.5) (end 133.5 164.5) (layer Cmts.User) (width 0.15))
   (gr_line (start 213.5 84.5) (end 133.5 84.5) (layer Cmts.User) (width 0.15))

Commit message: Utility and config changes
Parts:
- removed D2, D3, D4: 1N4007, Diode_THT:D_DO-35_SOD27_P2.54mm_Vertical_AnodeUp
- moved D1 45.1 mm to (174.3, 148.6)
- moved C2 0.64 mm to (171.8, 97.2)
Connections:
- J2 pad 5: Net-(D1-Pad2) -> Net-(D1-Pad1)
- R1 pad 1: Net-(D1-Pad1) -> Net-(R1-Pad1)
- U1 pad 1: Net-(D1-Pad1) -> Net-(R1-Pad1)
Routing:
- net Net-(D1-Pad2): track 128.5 -> 54.7 mm, vias 1 -> 0
- net Net-(D1-Pad1): track 54.8 -> 6.61 mm, vias 1 -> 0
- net Net-(R1-Pad1): track 0.00 -> 46.0 mm
- net Net-(R4-Pad1): track 66.2 -> 52.1 mm, vias 1 -> 0
- net Net-(R3-Pad1): track 63.5 -> 50.5 mm, vias 1 -> 0
- net Net-(R2-Pad1): track 61.4 -> 50.8 mm, vias 1 -> 0
- net Net-(C3-Pad1): track 247.8 -> 247.1 mm
- net Net-(C2-Pad2): track 8.43 -> 9.06 mm

Commit message: README...
Parts:
- removed the R11 at (177.5, 96.5)
- added R12: 100R, Resistor_THT:R_Axial_DIN0204_L3.6mm_D1.6mm_P5.08mm_Horizontal, F.Cu at (177.5, 96.5)
- J3: footprint TerminalBlock_Phoenix:TerminalBlock_Phoenix_MPT-0,5-4-2.54_1x04_P2.54mm_Horizontal -> TerminalBlock_Phoenix:TerminalBlock_Phoenix_MPT-0,5-5-2.54_1x05_P2.54mm_Horizontal
- JP1: value Jumper_NO_Small -> SCR; footprint Jumper:SolderJumper-3_P1.3mm_Open_Pad1.0x1.5mm -> Connector_PinHeader_2.54mm:PinHeader_1x02_P2.54mm_Vertical
- SW1: footprint Button_Switch_THT:SW_DIP_SPSTx08_Slide_6.7x21.88mm_W7.62mm_P2.54mm_LowProfile -> Package_DIP:DIP-14_W7.62mm
- moved JP1 3.89 mm to (183.8, 100.3), turned to 270 degrees
- moved J3 2.54 mm to (194.0, 94.0)
- moved SW1 0.64 mm to (168.6, 142.2)
- renumbered C4 to C1, C3 to C2, C1 to C3, C2 to C4, D5 to D2, D6 to D3, D7 to D4, D8 to D5, D9 to D6, R13 to R1, R9 to R10, R10 to R11, R12 to R13, R1 to R2, R2 to R3, R3 to R4, R4 to R5, R5 to R6, R6 to R7, R7 to R8, R8 to R9
Connections:
- JP1 pad 2: Net-(J3-Pad2) -> Net-(J3-Pad5)
- SW1 pad 8: GND -> Net-(SW1-Pad8)
- U2 pad 15: Net-(SW1-Pad16) -> (no net)
- U2 pad 16: Net-(SW1-Pad15) -> Net-(SW1-Pad14)
- U2 pad 17: Net-(SW1-Pad14) -> Net-(SW1-Pad13)
- U2 pad 18: Net-(SW1-Pad13) -> Net-(SW1-Pad12)
- U2 pad 19: Net-(SW1-Pad12) -> Net-(SW1-Pad11)
- U2 pad 20: Net-(SW1-Pad11) -> Net-(SW1-Pad10)
- U2 pad 21: Net-(SW1-Pad10) -> Net-(SW1-Pad9)
- U2 pad 22: Net-(SW1-Pad9) -> Net-(SW1-Pad8)
Routing:
- net Net-(J3-Pad5): track 0.00 -> 7.40 mm
- net Net-(J3-Pad2): track 27.6 -> 20.4 mm
- net Net-(SW1-Pad16): track 6.92 -> 0.00 mm
- net Net-(SW1-Pad15): track 6.92 -> 0.00 mm
- net Net-(SW1-Pad8): track 0.00 -> 5.61 mm
- net Net-(J3-Pad4): track 18.5 -> 21.7 mm
- net Net-(J3-Pad3): track 23.8 -> 26.4 mm
- net Net-(F2-Pad1): track 18.1 -> 15.5 mm
- net Net-(SW1-Pad10): track 6.92 -> 5.61 mm
- net Net-(SW1-Pad14): track 6.92 -> 5.61 mm
- net Net-(SW1-Pad11): track 6.92 -> 5.61 mm
- net Net-(SW1-Pad9): track 6.92 -> 5.61 mm
- net Net-(SW1-Pad13): track 6.92 -> 5.61 mm
- net Net-(SW1-Pad12): track 6.92 -> 5.61 mm
Other:
- board text added: "16"
- board text added: "32"
- board text added: "64"
- board text added: "8"
- board text added: "SCR"
- board text removed: "3"
- board text removed: "5"
- board text removed: "6"
- board text removed: "7"
