File: modules/winint/hardware/1.0/kicad/modint-v1.0.sch (KiCad schematic (older format))
At the start: 39 parts, among them J1 NPN SENSOR, J2 Screw_Terminal_01x05, J3 M12-5PIN, J4 RELAYS, K1 SANYOU_SRD_Form_C, K2 SANYOU_SRD_Form_C, Q1 2N2219, Q2 2N2219, SW1 INSTANCE, U1 CNY74-4H, U2 Teensy_3.2, U3 TEC2-2411WI, U4 MCP2551-I-P

Commit message: Refactor
Changed lines of the file:
@@
 	2450 850  2450 3350
 Wire Wire Line
-	5150 1750 5050 1750
+	5550 1750 5050 1750
 Wire Wire Line
-	5150 850  5150 1750
+	5550 850  5550 1750
 Wire Wire Line
 	5350 1650 5050 1650
@@
 	5050 1450 5250 1450
 Wire Wire Line
-	2950 1150 5450 1150
+	2950 1150 5150 1150
 Wire Wire Line
-	5450 1150 5450 1350
+	5150 1150 5150 1350
 Wire Wire Line
-	5450 1350 5050 1350
+	5150 1350 5050 1350
 Wire Wire Line
 	10150 1500 9900 1500
@@
 	1850 750  3050 750
 Wire Wire Line
-	2450 850  5150 850
+	2450 850  5550 850
 Wire Wire Line
 	3950 2650 3850 2650
