File: modules/winint/hardware/1.0/kicad/winint-1.0.sch (KiCad schematic (older format))
At the start: 66 parts, among them J1 ROT, J2 RET, J3 DEP, J4 RTG, J5 DPG, J6 OVL, J7 Screw_Terminal_01x03, J8 Screw_Terminal_01x03, J9 Screw_Terminal_01x05, K1 RS_476-257, K2 RS_476-257, Q1 NTE123A, Q2 NTE123A, SW1 CONFIG, SW2 INSTANCE, U1 PC817, U2 PC817, U3 PC817, U4 PC817, U5 PC817, U6 PC817, U7 Teensy_3.2, U8 MCP2551-I-P, U9 TEC2-2411WI

Commit message: Tidy up
Parts:
- D1, D4, D5: value DOWN -> FA3863X
- D2: value UP -> FA3863X
- D3: value PWR/TX -> FA3863X
- J7: value Screw_Terminal_01x03 -> UP
- J8: value Screw_Terminal_01x03 -> DOWN
- J9: value Screw_Terminal_01x05 -> CAN
Other:
- moved on the sheet: C1
Changed lines of the file:
@@
 F 1 "1A" V 9400 3250 39  0000 C CNN
 F 2 "Fuse:Fuse_Littelfuse_395Series" H 9500 2900 50  0001 L CNN
-F 3 "~" H 9450 3100 50  0001 C CNN
+F 3 "https://docs.rs-online.com/ec39/0900766b80bc9043.pdf" H 9450 3100 50  0001 C CNN
 	1    9450 3100
 	0    1    1    0
@@
 U 1 1 5F3B6D27
 P 9600 6300
-F 0 "D3" H 9650 6200 50  0000 R CNN
-F 1 "PWR/TX" H 9400 6250 39  0001 R CNN
+F 0 "D3" H 9600 6200 50  0000 C CNN
+F 1 "FA3863X" H 9600 6400 39  0000 C CNN
 F 2 "LED_THT:LED_D3.0mm" H 9600 6300 50  0001 C CNN
-F 3 "~" H 9600 6300 50  0001 C CNN
+F 3 "https://docs.rs-online.com/4848/0900766b80f2cc5c.pdf" H 9600 6300 50  0001 C CNN
 	1    9600 6300
 	-1   0    0    1
@@
 L Device:C C1
 U 1 1 5F38A0E7
-P 3950 6550
-F 0 "C1" V 4000 6500 50  0000 R CNN
-F 1 "100nF" V 3900 6500 39  0000 R CNN
-F 2 "Capacitor_THT:CP_Radial_D5.0mm_P2.50mm" H 3988 6400 50  0001 C CNN
-F 3 "~" H 3950 6550 50  0001 C CNN
-	1    3950 6550
+P 3950 6600
+F 0 "C1" V 4000 6550 50  0000 R CNN
+F 1 "100nF" V 3900 6550 39  0000 R CNN
+F 2 "Capacitor_THT:CP_Radial_D5.0mm_P2.50mm" H 3988 6450 50  0001 C CNN
+F 3 "~" H 3950 6600 50  0001 C CNN
+	1    3950 6600
 	0    -1   -1   0
 $EndComp
@@
 U 1 1 5F60BF0B
 P 2600 5450
-F 0 "SW2" H 2600 6117 50  0000 C CNN
-F 1 "INSTANCE" H 2600 6026 50  0000 C CNN
+F 0 "SW2" H 2600 6000 50  0000 C CNN
+F 1 "INSTANCE" H 2600 5100 50  0000 C CNN
 F 2 "Button_Switch_THT:SW_DIP_SPSTx07_Slide_6.7x19.34mm_W7.62mm_P2.54mm_LowProfile" H 2600 5450 50  0001 C CNN
 F 3 "~" H 2600 5450 50  0001 C CNN
@@
 U 1 1 5F2F9489
 P 4500 6250
-F 0 "U7" H 5450 4800 50  0000 C CNN
-F 1 "Teensy_3.2" H 5050 6250 50  0000 C CNN
+F 0 "U7" H 5050 4800 50  0000 C CNN
+F 1 "Teensy_3.2" H 5050 6400 50  0000 C CNN
 F 2 "PDJR:Teensy30_31_32_LC" H 4500 6250 50  0001 C CNN
 F 3 "" H 4500 6250 50  0001 C CNN
@@
 $EndComp
 Wire Wire Line
-	4100 6550 4600 6550
+	4100 6600 4600 6600
 Wire Wire Line
 	3400 6150 3100 6150
@@
 	3400 6250 3300 6250
 Wire Wire Line
-	3300 6550 3800 6550
-Wire Wire Line
-	4600 6550 4600 6250
+	3300 6600 3800 6600
+Wire Wire Line
+	4600 6600 4600 6250
 Wire Wire Line
 	4600 6250 4500 6250
@@
 U 1 1 6069075F
 P 10700 3300
-F 0 "J9" H 10780 3342 50  0000 L CNN
-F 1 "Screw_Terminal_01x05" H 10780 3251 50  0000 L CNN
+F 0 "J9" H 10650 3600 50  0000 L CNN
+F 1 "CAN" H 10700 3000 50  0000 C CNN
 F 2 "TerminalBlock_Phoenix:TerminalBlock_Phoenix_MPT-0,5-5-2.54_1x05_P2.54mm_Horizontal" H 10700 3300 50  0001 C CNN
 F 3 "~" H 10700 3300 50  0001 C CNN
@@
 U 1 1 600EA741
 P 9600 5900
-F 0 "D2" H 9650 5800 50  0000 R CNN
-F 1 "UP" H 9400 5850 39  0001 R CNN
+F 0 "D2" H 9600 5800 50  0000 C CNN
+F 1 "FA3863X" H 9600 6000 39  0000 C CNN
 F 2 "LED_THT:LED_D3.0mm" H 9600 5900 50  0001 C CNN
-F 3 "~" H 9600 5900 50  0001 C CNN
+F 3 "https://docs.rs-online.com/4848/0900766b80f2cc5c.pdf" H 9600 5900 50  0001 C CNN
 	1    9600 5900
 	-1   0    0    1
@@
 U 1 1 5FBEC238
 P 10700 1200
-F 0 "J7" H 10780 1242 50  0000 L CNN
-F 1 "Screw_Terminal_01x03" H 10780 1151 50  0000 L CNN
+F 0 "J7" H 10650 1400 50  0000 L CNN
+F 1 "UP" H 10650 1000 50  0000 L CNN
 F 2 "TerminalBlock_Phoenix:TerminalBlock_Phoenix_MPT-0,5-3-2.54_1x03_P2.54mm_Horizontal" H 10700 1200 50  0001 C CNN
 F 3 "~" H 10700 1200 50  0001 C CNN
@@
 U 1 1 5FCE91C6
 P 10700 2300
-F 0 "J8" H 10780 2342 50  0000 L CNN
-F 1 "Screw_Terminal_01x03" H 10780 2251 50  0000 L CNN
+F 0 "J8" H 10650 2500 50  0000 L CNN
+F 1 "DOWN" H 10600 2100 50  0000 L CNN
 F 2 "TerminalBlock_Phoenix:TerminalBlock_Phoenix_MPT-0,5-3-2.54_1x03_P2.54mm_Horizontal" H 10700 2300 50  0001 C CNN
 F 3 "~" H 10700 2300 50  0001 C CNN
@@
 P 7950 1400
 F 0 "D4" V 7950 1250 50  0000 L CNN
-F 1 "DOWN" H 7650 1350 39  0001 C CNN
+F 1 "FA3863X" V 7850 1400 39  0000 C CNN
 F 2 "Connector_PinHeader_2.54mm:PinHeader_1x02_P2.54mm_Vertical" H 7950 1400 50  0001 C CNN
-F 3 "~" H 7950 1400 50  0001 C CNN
+F 3 "https://docs.rs-online.com/4848/0900766b80f2cc5c.pdf" H 7950 1400 50  0001 C CNN
 	1    7950 1400
 	0    -1   -1   0
@@
 U 1 1 5FC4BE6B
 P 7950 2100
-F 0 "R22" H 8050 2100 50  0000 C CNN
+F 0 "R22" H 8150 2100 50  0000 R CNN
 F 1 "200R" V 7950 2100 39  0000 C CNN
 F 2 "Resistor_THT:R_Axial_DIN0204_L3.6mm_D1.6mm_P5.08mm_Horizontal" V 7880 2100 50  0001 C CNN
@@
 P 7950 2500
 F 0 "D5" V 7950 2450 50  0000 R CNN
-F 1 "DOWN" H 7650 2450 39  0001 C CNN
+F 1 "FA3863X" V 7850 2500 39  0000 C CNN
 F 2 "Connector_PinHeader_2.54mm:PinHeader_1x02_P2.54mm_Vertical" H 7950 2500 50  0001 C CNN
-F 3 "~" H 7950 2500 50  0001 C CNN
+F 3 "https://docs.rs-online.com/4848/0900766b80f2cc5c.pdf" H 7950 2500 50  0001 C CNN
 	1    7950 2500
 	0    -1   -1   0
@@
 L Switch:SW_DIP_x02 SW1
 U 1 1 5FD67EF1
-P 2600 4450
-F 0 "SW1" H 2600 4817 50  0000 C CNN
-F 1 "CONFIG" H 2600 4726 50  0000 C CNN
-F 2 "Button_Switch_THT:SW_DIP_SPSTx02_Slide_6.7x6.64mm_W7.62mm_P2.54mm_LowProfile" H 2600 4450 50  0001 C CNN
-F 3 "~" H 2600 4450 50  0001 C CNN
-	1    2600 4450
-	1    0    0    -1
-$EndComp
-Text Label 2900 4350 0    50   ~ 0
+P 2600 4350
+F 0 "SW1" H 2600 4200 50  0000 C CNN
+F 1 "CONFIG" H 2600 4600 50  0000 C CNN
+F 2 "Button_Switch_THT:SW_DIP_SPSTx02_Slide_6.7x6.64mm_W7.62mm_P2.54mm_LowProfile" H 2600 4350 50  0001 C CNN
+F 3 "~" H 2600 4350 50  0001 C CNN
+	1    2600 4350
+	1    0    0    1
+$EndComp
+Text Label 2900 4450 0    50   ~ 0
 CAN_SCR
 Wire Wire Line
@@
 Connection ~ 2300 5650
 Wire Wire Line
-	3300 6250 3300 6550
+	3300 6250 3300 6600
 $Comp
 L power:GND #PWR02
@@
 $EndComp
 Wire Wire Line
-	3300 6650 3300 6550
-Connection ~ 3300 6550
+	3300 6650 3300 6600
+Connection ~ 3300 6600
 $Comp
 L power:GND #PWR016
@@
 $EndComp
 Wire Wire Line
-	4600 6650 4600 6550
-Connection ~ 4600 6550
+	4600 6650 4600 6600
+Connection ~ 4600 6600
 Wire Wire Line
 	6800 1200 6950 1200
@@
 Text Label 6800 2300 2    50   ~ 0
 RELAY_DOWN
-Wire Wire Line
-	2300 5050 2300 4450
 Connection ~ 2300 5050
 Text Label 4500 4950 0    50   ~ 0
@@
 Wire Wire Line
 	2700 3450 3100 3450
-Text Label 2900 4450 0    50   ~ 0
+Text Label 2900 4350 0    50   ~ 0
 ENABLE
 Text Label 4500 6150 0    50   ~ 0
@@
 U 1 1 600EA320
 P 9600 5500
-F 0 "D1" H 9650 5400 50  0000 R CNN
-F 1 "DOWN" H 9400 5450 39  0001 R CNN
+F 0 "D1" H 9600 5400 50  0000 C CNN
+F 1 "FA3863X" H 9600 5600 39  0000 C CNN
 F 2 "LED_THT:LED_D3.0mm" H 9600 5500 50  0001 C CNN
-F 3 "~" H 9600 5500 50  0001 C CNN
+F 3 "https://docs.rs-online.com/4848/0900766b80f2cc5c.pdf" H 9600 5500 50  0001 C CNN
 	1    9600 5500
 	-1   0    0    1
@@
 CAN_SCR
 Wire Wire Line
-	2300 4450 2300 4350
+	2300 4350 2300 4450
 Connection ~ 2300 4450
+Wire Wire Line
+	2300 4450 2300 5050
 $EndSCHEMATC
