File: modules/winint/hardware/1.0/kicad/winint-1.0.kicad_pcb (KiCad board)
At the start: 2 copper layers, 75 x 75 mm, 70 parts, among them J1 ROT, J2 RET, J3 DEP, J4 RTG, J5 DPG, J6 OVL, J7 Screw_Terminal_01x03, J8 Screw_Terminal_01x03, J9 Screw_Terminal_01x05, K1 RS_476-257, K2 RS_476-257, Q1 NTE123A, Q2 NTE123A, SW1 CONFIG, SW2 INSTANCE, U1 PC817, U2 PC817, U3 PC817, U4 PC817, U5 PC817, U6 PC817, U7 Teensy_3.2, U8 MCP2551-I-P, U9 TEC2-2411WI

Commit message: Tweak
Parts:
- D3: renamed from De; value PWR -> PWR/TX
Connections:
- net /CANH renamed /CAN_H
- net /CANL renamed /CAN_L
- net /CANSCR renamed /CAN_SCR

Commit message: Tidy
Connections:
- net /NETC renamed /NET_C
- net /NETS renamed /NET_S

Commit message: Build system prep
Parts:
- D1, D4, D5: value DOWN -> L-1334SRT
- D2: value UP -> L-1334SRT
- D3: value PWR/TX -> L-1334SRT
- J7: value Screw_Terminal_01x03 -> UP
- J8: value Screw_Terminal_01x03 -> DOWN
- J9: value Screw_Terminal_01x05 -> CAN
- K1, K2: value RS_476-257 -> 476-757
Changed lines of the file:
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@@
     (add_net "Net-(SW2-Pad8)")
     (add_net "Net-(SW2-Pad9)")
+    (add_net "Net-(U7-Pad12)")
+    (add_net "Net-(U7-Pad13)")
+    (add_net "Net-(U7-Pad15)")
+    (add_net "Net-(U7-Pad26)")
+    (add_net "Net-(U8-Pad5)")
+    (add_net "Net-(U9-Pad3)")
+    (add_net "Net-(U9-Pad5)")
+    (add_net "Net-(U9-Pad8)")
   )
   (module Package_DIP:DIP-4_W7.62mm (layer F.Cu)
@@
       (effects (font (size 1 1) (thickness 0.15)))
     )
-    (fp_text value Screw_Terminal_01x03 (at 2.54 4.16 180) (layer F.Fab)
+    (fp_text value UP (at 2.54 4.16 180) (layer F.Fab)
       (effects (font (size 1 1) (thickness 0.15)))
     )
@@
       (effects (font (size 1 1) (thickness 0.15)))
     )
-    (fp_text value DOWN (at 0 4.87 90) (layer F.Fab)
+    (fp_text value L-1334SRT (at 0 4.87 90) (layer F.Fab)
       (effects (font (size 1 1) (thickness 0.15)))
     )
@@
       (effects (font (size 1 1) (thickness 0.15)))
     )
-    (fp_text value DOWN (at 0 4.87 90) (layer F.Fab)
+    (fp_text value L-1334SRT (at 0 4.87 90) (layer F.Fab)
       (effects (font (size 1 1) (thickness 0.15)))
     )
@@
       (effects (font (size 1 1) (thickness 0.15)))
     )
-    (fp_text value Screw_Terminal_01x05 (at 5.08 4.16) (layer F.Fab)
+    (fp_text value CAN (at 5.08 4.16) (layer F.Fab)
       (effects (font (size 1 1) (thickness 0.15)))
     )
@@
       (effects (font (size 1 1) (thickness 0.15)))
     )
-    (fp_text value Screw_Terminal_01x03 (at 2.54 4.16) (layer F.Fab)
+    (fp_text value DOWN (at 2.54 4.16) (layer F.Fab)
       (effects (font (size 1 1) (thickness 0.15)))
     )
@@
       (effects (font (size 1 1) (thickness 0.15)))
     )
-    (fp_text value DOWN (at 1.143 2.413 180) (layer F.SilkS)
+    (fp_text value L-1334SRT (at 1.143 2.413 180) (layer F.SilkS)
       (effects (font (size 1 1) (thickness 0.15)) (justify right))
     )
@@
       (effects (font (size 1 1) (thickness 0.15)))
     )
-    (fp_text value RS_476-257 (at 0 5.08 90) (layer F.Fab)
+    (fp_text value 476-757 (at 0 5.08 90) (layer F.Fab)
       (effects (font (size 1 1) (thickness 0.15)))
     )
@@
       (effects (font (size 1 1) (thickness 0.15)))
     )
-    (fp_text value RS_476-257 (at 0 5.08 90) (layer F.Fab)
+    (fp_text value 476-757 (at 0 5.08 90) (layer F.Fab)
       (effects (font (size 1 1) (thickness 0.15)))
     )
@@
       (effects (font (size 1 1) (thickness 0.15)))
     )
-    (fp_text value UP (at 1.27 2.413 180) (layer F.SilkS)
+    (fp_text value L-1334SRT (at 1.27 2.413 180) (layer F.SilkS)
       (effects (font (size 1 1) (thickness 0.15)) (justify right))
     )
@@
       (effects (font (size 1 1) (thickness 0.15)))
     )
-    (fp_text value PWR/TX (at 1.143 2.413 180) (layer F.SilkS)
+    (fp_text value L-1334SRT (at 1.143 2.413 180) (layer F.SilkS)
       (effects (font (size 1 1) (thickness 0.15)) (justify right))
     )
@@
   (segment (start 183.185 107.315) (end 181.915 106.045) (width 1) (layer B.Cu) (net 17))
   (segment (start 183.185 109.22) (end 183.185 107.315) (width 1) (layer B.Cu) (net 17))
-  (segment (start 206.68 88.9) (end 207.95 90.17) (width 1) (layer B.Cu) (net 66))
-  (segment (start 166.675 88.9) (end 206.68 88.9) (width 1) (layer B.Cu) (net 66))
-  (segment (start 163.5 93.98) (end 163.5 92.075) (width 1) (layer B.Cu) (net 66))
-  (segment (start 163.5 92.075) (end 166.675 88.9) (width 1) (layer B.Cu) (net 66))
-  (segment (start 164.135 88.9) (end 160.96 92.075) (width 1) (layer F.Cu) (net 67))
-  (segment (start 201.6 88.9) (end 164.135 88.9) (width 1) (layer F.Cu) (net 67))
-  (segment (start 160.96 92.075) (end 160.96 93.98) (width 1) (layer F.Cu) (net 67))
-  (segment (start 205.41 104.14) (end 205.41 92.71) (width 1) (layer F.Cu) (net 67))
-  (segment (start 205.41 92.71) (end 201.6 88.9) (width 1) (layer F.Cu) (net 67))
   (segment (start 167.31 150.495) (end 166.04 149.225) (width 0.5) (layer B.Cu) (net 18))
   (segment (start 167.31 154.94) (end 167.31 150.495) (width 0.5) (layer B.Cu) (net 18))
@@
   (segment (start 161.595 97.79) (end 159.69 99.695) (width 0.5) (layer B.Cu) (net 65))
   (segment (start 169.215 97.79) (end 161.595 97.79) (width 0.5) (layer B.Cu) (net 65))
+  (segment (start 206.68 88.9) (end 207.95 90.17) (width 1) (layer B.Cu) (net 66))
+  (segment (start 166.675 88.9) (end 206.68 88.9) (width 1) (layer B.Cu) (net 66))
+  (segment (start 163.5 93.98) (end 163.5 92.075) (width 1) (layer B.Cu) (net 66))
+  (segment (start 163.5 92.075) (end 166.675 88.9) (width 1) (layer B.Cu) (net 66))
+  (segment (start 164.135 88.9) (end 160.96 92.075) (width 1) (layer F.Cu) (net 67))
+  (segment (start 201.6 88.9) (end 164.135 88.9) (width 1) (layer F.Cu) (net 67))
+  (segment (start 160.96 92.075) (end 160.96 93.98) (width 1) (layer F.Cu) (net 67))
+  (segment (start 205.41 104.14) (end 205.41 92.71) (width 1) (layer F.Cu) (net 67))
+  (segment (start 205.41 92.71) (end 201.6 88.9) (width 1) (layer F.Cu) (net 67))
   (zone (net 2) (net_name GND) (layer F.Cu) (hatch edge 0.508)
     (connect_pads (clearance 0.508))
     (min_thickness 0.254)
-    (fill yes (arc_segments 32) (thermal_gap 0.508) (thermal_bridge_width 0.508))
+    (fill (arc_segments 32) (thermal_gap 0.508) (thermal_bridge_width 0.508))
     (polygon
       (pts
@@
     (connect_pads (clearance 0.508))
     (min_thickness 0.254)
-    (fill yes (arc_segments 32) (thermal_gap 0.508) (thermal_bridge_width 0.508))
+    (fill (arc_segments 32) (thermal_gap 0.508) (thermal_bridge_width 0.508))
     (polygon
       (pts
