File: modules/winctl/hardware/1.0/kicad/winctl-1.0.sch (KiCad schematic (older format))
At the start: 39 parts, among them J1 SWITCH INPUTS, J2 RELAY OUTPUTS, J3 M12-5PIN, SW1 PRGW0, SW2 PRGW1, SW3 INSTANCE, U1 POWER, U2 W0UP, U3 CNY74-4H, U4 W0DN, U5 W1UP, U6 W1DN, U7 Teensy_3.2, U8 TEC2-2411WI, U9 MCP2551-I-P

Commit message: Refactor
Changed lines of the file:
@@
 encoding utf-8
 Sheet 1 1
-Title "WCTRL - windlass control interface module"
+Title "WINCTL - windlass control interface module"
 Date "2020-09-14"
-Rev "V1.0"
+Rev "1.0"
 Comp "PDJR <preeve@pdjr.eu>"
 Comment1 ""
@@
 Connection ~ 8450 2550
 Wire Wire Line
-	9050 2550 9450 2550
+	9050 2550 9400 2550
 Connection ~ 9050 2550
 Connection ~ 7850 1500
@@
 Connection ~ 8800 6200
 Wire Wire Line
-	8800 6200 9450 6200
+	8800 6200 9400 6200
 Wire Wire Line
 	8050 3050 8250 3050
@@
 	1    0    0    -1
 $EndComp
-Connection ~ 9450 6200
+Connection ~ 9400 6200
 Wire Wire Line
 	8050 3050 8050 3350
@@
 	8150 1900 8150 3550
 Wire Wire Line
-	9450 6200 9600 6200
+	9400 6200 9600 6200
 Wire Wire Line
 	9700 1900 9700 2850
@@
 	9700 2850 9950 2850
 Wire Wire Line
-	9450 2550 9450 6200
+	9400 2550 9400 6200
 Wire Wire Line
 	9250 1900 9700 1900

Commit message: Revised PCB
Parts:
- removed JP1: 2-4, Connector_PinHeader_2.54mm:PinHeader_1x02_P2.54mm_Vertical, symbol Jumper:Jumper_2_Open
- removed JP2: 2-6, Connector_PinHeader_2.54mm:PinHeader_1x02_P2.54mm_Vertical, symbol Jumper:Jumper_2_Open
- removed JP3: 2-8, Connector_PinHeader_2.54mm:PinHeader_1x02_P2.54mm_Vertical, symbol Jumper:Jumper_2_Open
- removed JP4: 2-10, Connector_PinHeader_2.54mm:PinHeader_1x02_P2.54mm_Vertical, symbol Jumper:Jumper_2_Open
- removed SW1: PRGW0, Button_Switch_THT:KSA_Tactile_SPST, symbol Switch:SW_Push
- removed SW2: PRGW1, Button_Switch_THT:KSA_Tactile_SPST, symbol Switch:SW_Push
- added Q1, Q2, Q3, Q4, Q5: 2N7000, Package_TO_SOT_THT:TO-92_Inline, symbol Transistor_FET:2N7000
- added R1, R10, R11, R12, R13, R14, R2, R7, R8, R9: 10K, Resistor_THT:R_Axial_DIN0207_L6.3mm_D2.5mm_P2.54mm_Vertical, symbol Device:R
- added SW1: PRG0, Button_Switch_THT:SW_TH_Tactile_Omron_B3F-10xx, symbol PDJR:SW_Push
- added SW2: PRG1, Button_Switch_THT:SW_TH_Tactile_Omron_B3F-10xx, symbol PDJR:SW_Push
- renumbered R5 to R15, R6 to R16, R7 to R17, R8 to R18, R9 to R19, R10 to R20, R1 to R3, R2 to R4, R3 to R5, R4 to R6
Connections:
- wire segments 214 -> 247
- no-connect marks 5 -> 4
Other:
- moved on the sheet: J2

Commit message: Revised PCB
Connections:
- net GND: now also U7.27 (AGND)
- net at J1.2 (Pin_2): now also R4.1; no longer R4.2
- net at U3.4: now also R4.2; no longer R4.1
- net at J2.2 (Pin_2): now also U1.7; no longer U2.1
- net at J2.3 (Pin_3): now also U2.1; no longer U4.1
- net at J2.4 (Pin_4): now also U2.7; no longer U5.1
- net at J2.5 (Pin_5): now also U4.1; no longer U6.1
- net at J2.6 (Pin_6): now also U4.7; no longer U1.7
- net at J2.7 (Pin_7): now also U5.1; no longer U2.7
- net at J2.8 (Pin_8): now also U5.7; no longer U4.7
- net at J2.9 (Pin_9): now also U6.1; no longer U5.7
- no-connect marks 4 -> 3
Changed lines of the file:
@@
 Sheet 1 1
 Title "WINCTL - windlass control interface module"
-Date "2020-09-14"
-Rev "1.0"
+Date "2020-10-17"
+Rev "1.1"
 Comp "PDJR <preeve@pdjr.eu>"
 Comment1 ""
@@
 F 4 "1W" V 2350 2650 50  0001 C CNN "Power"
 	1    2350 2650
-	0    1    1    0
+	0    -1   -1   0
 $EndComp
 $Comp
@@
 Connection ~ 4900 4850
 Wire Wire Line
-	4900 4850 6500 4850
+	4900 4850 5100 4850
 Wire Wire Line
 	6700 3650 6900 3650
@@
 Wire Wire Line
 	7200 3750 7500 3750
-NoConn ~ 5300 3650
 Connection ~ 8150 3650
 Wire Wire Line
@@
 Wire Wire Line
 	3800 4750 4250 4750
-Wire Wire Line
-	3050 5950 3850 5950
-Wire Wire Line
-	3850 5950 3850 5450
-Wire Wire Line
-	2950 5850 3400 5850
-Wire Wire Line
-	3400 5850 3400 5450
-Wire Wire Line
-	2850 5750 2950 5750
-Wire Wire Line
-	2950 5750 2950 5450
-Wire Wire Line
-	2750 5850 2500 5850
-Wire Wire Line
-	2500 5850 2500 5450
-Wire Wire Line
-	2650 6900 2650 5950
-Wire Wire Line
-	2650 5950 2050 5950
-Wire Wire Line
-	2050 5950 2050 5450
-Wire Wire Line
-	3150 6900 3150 6050
-Wire Wire Line
-	3150 6050 2350 6050
-Wire Wire Line
-	2350 6050 2350 5450
-Wire Wire Line
-	3250 6900 3250 5650
-Wire Wire Line
-	3250 5650 2800 5650
-Wire Wire Line
-	2800 5650 2800 5450
-Wire Wire Line
-	3350 6900 3350 5550
-Wire Wire Line
-	3350 5550 3250 5550
-Wire Wire Line
-	3250 5550 3250 5450
-Wire Wire Line
-	3450 6900 3450 6050
-Wire Wire Line
-	3700 6050 3700 5450
-Wire Wire Line
-	3450 6050 3700 6050
-Wire Wire Line
-	3550 6900 3550 6150
-Wire Wire Line
-	3550 6150 4150 6150
-Wire Wire Line
-	4150 6150 4150 5450
-Wire Wire Line
-	2750 5850 2750 6900
-Wire Wire Line
-	2850 5750 2850 6900
-Wire Wire Line
-	2950 5850 2950 6900
-Wire Wire Line
-	3050 5950 3050 6900
 $Comp
 L PDJR:SW_Push SW1
@@
 	0    1    -1   0
 $EndComp
+Wire Wire Line
+	3050 6900 3050 6050
+Wire Wire Line
+	3050 6050 2950 6050
+Wire Wire Line
+	2950 6050 2950 5450
+Wire Wire Line
+	3150 6900 3150 6050
+Wire Wire Line
+	3150 6050 3250 6050
+Wire Wire Line
+	3250 6050 3250 5450
+Wire Wire Line
+	3250 6900 3250 6150
+Wire Wire Line
+	3250 6150 3400 6150
+Wire Wire Line
+	3400 6150 3400 5450
+Wire Wire Line
+	3350 6900 3350 6250
+Wire Wire Line
+	3350 6250 3700 6250
+Wire Wire Line
+	3700 6250 3700 5450
+Wire Wire Line
+	3450 6900 3450 6350
+Wire Wire Line
+	3450 6350 3850 6350
+Wire Wire Line
+	3850 6350 3850 5450
+Wire Wire Line
+	3550 6900 3550 6450
+Wire Wire Line
+	3550 6450 4150 6450
+Wire Wire Line
+	4150 6450 4150 5450
+Wire Wire Line
+	2950 6900 2950 6150
+Wire Wire Line
+	2950 6150 2800 6150
+Wire Wire Line
+	2800 6150 2800 5450
+Wire Wire Line
+	2850 6900 2850 6250
+Wire Wire Line
+	2850 6250 2500 6250
+Wire Wire Line
+	2500 6250 2500 5450
+Wire Wire Line
+	2750 6900 2750 6350
+Wire Wire Line
+	2750 6350 2350 6350
+Wire Wire Line
+	2350 6350 2350 5450
+Wire Wire Line
+	2650 6900 2650 6450
+Wire Wire Line
+	2650 6450 2050 6450
+Wire Wire Line
+	2050 6450 2050 5450
+Wire Wire Line
+	5300 3650 5100 3650
+Wire Wire Line
+	5100 3650 5100 4850
+Connection ~ 5100 4850
+Wire Wire Line
+	5100 4850 6500 4850
 $EndSCHEMATC
