File: modules/winctl/hardware/1.0/kicad/winctl-1.0.kicad_pcb (KiCad board)
At the start: 2 copper layers, 75 x 75 mm, 43 parts, among them J1 SWITCH INPUTS, J2 RELAY OUTPUTS, J3 M12-5PIN, SW1 PRGW0, SW2 PRGW1, SW3 INSTANCE, U1 POWER, U2 W0UP, U3 CNY74-4H, U4 W0DN, U5 W1UP, U6 W1DN, U7 Teensy_3.2, U8 TEC2-2411WI, U9 MCP2551-I-P

Commit message: Refactor
Other:
- board text added: "WINCTL 1.0"
- board text removed: "WCTL 1.0"
Changed lines of the file:
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@@
   )
   (page A4)
+  (title_block
+    (title "WINCTL - windlass control interface module")
+    (date 2020-09-15)
+    (rev 1.0)
+    (company PDJR)
+  )
   (layers
-    (0 F.Cu signal)
-    (31 B.Cu signal)
+    (0 F.Cu signal hide)
+    (31 B.Cu signal hide)
     (33 F.Adhes user hide)
     (35 F.Paste user hide)
@@
     (add_net "Net-(U5-Pad3)")
     (add_net "Net-(U6-Pad3)")
+    (add_net "Net-(U7-Pad15)")
+    (add_net "Net-(U7-Pad26)")
+    (add_net "Net-(U7-Pad27)")
     (add_net "Net-(U7-Pad5)")
     (add_net "Net-(U7-Pad6)")
+    (add_net "Net-(U8-Pad3)")
+    (add_net "Net-(U8-Pad5)")
+    (add_net "Net-(U8-Pad8)")
+    (add_net "Net-(U9-Pad5)")
   )
   (module Connector_PinHeader_2.54mm:PinHeader_1x02_P2.54mm_Vertical (layer F.Cu)
@@
     (effects (font (size 2 1.5) (thickness 0.3)) (justify left))
   )
-  (gr_text "WCTL 1.0" (at 38.735 86.36) (layer F.SilkS)
+  (gr_text "WINCTL 1.0" (at 35.56 86.36) (layer F.SilkS)
     (effects (font (size 3 2) (thickness 0.3)) (justify left))
   )

Commit message: Gerber order to ELecrow
Other:
- board text added: "Sep 2020"
Changed lines of the file:
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@@
   (general
     (thickness 1.6)
-    (drawings 120)
+    (drawings 121)
     (tracks 322)
     (zones 0)
@@
     (35 F.Paste user hide)
     (37 F.SilkS user)
-    (38 B.Mask user)
-    (39 F.Mask user)
+    (38 B.Mask user hide)
+    (39 F.Mask user hide)
     (40 Dwgs.User user hide)
     (41 Cmts.User user hide)
@@
     (visible_elements FFFFFF7F)
     (pcbplotparams
-      (layerselection 0x010e8_ffffffff)
+      (layerselection 0x010e0_ffffffff)
       (usegerberextensions true)
       (usegerberattributes false)
@@
     (add_net "Net-(U5-Pad3)")
     (add_net "Net-(U6-Pad3)")
-    (add_net "Net-(U7-Pad15)")
-    (add_net "Net-(U7-Pad26)")
-    (add_net "Net-(U7-Pad27)")
     (add_net "Net-(U7-Pad5)")
     (add_net "Net-(U7-Pad6)")
-    (add_net "Net-(U8-Pad3)")
-    (add_net "Net-(U8-Pad5)")
-    (add_net "Net-(U8-Pad8)")
-    (add_net "Net-(U9-Pad5)")
   )
   (module Connector_PinHeader_2.54mm:PinHeader_1x02_P2.54mm_Vertical (layer F.Cu)
@@
     )
   )
+  (gr_text "Sep 2020" (at 35 86.995) (layer F.SilkS)
+    (effects (font (size 2 1.5) (thickness 0.3)) (justify left))
+  )
   (gr_circle (center 44 79.295) (end 50 79.295) (layer Cmts.User) (width 0.15))
   (gr_circle (center 44 79.135) (end 50 79.135) (layer Cmts.User) (width 0.15))
@@
     (effects (font (size 2 1.5) (thickness 0.3)) (justify left))
   )
-  (gr_text "WINCTL 1.0" (at 35.56 86.36) (layer F.SilkS)
-    (effects (font (size 3 2) (thickness 0.3)) (justify left))
+  (gr_text "WINCTL 1.0" (at 35 83.5) (layer F.SilkS)
+    (effects (font (size 2 1.5) (thickness 0.3)) (justify left))
   )
   (gr_text "NMEA 2000 Windlass Control Interface Module" (at -17.78 27.305) (layer Eco1.User)

Commit message: Revised PCB
Parts:
- removed JP1: 2-4, Connector_PinHeader_2.54mm:PinHeader_1x02_P2.54mm_Vertical
- removed JP2: 2-6, Connector_PinHeader_2.54mm:PinHeader_1x02_P2.54mm_Vertical
- removed JP3: 2-8, Connector_PinHeader_2.54mm:PinHeader_1x02_P2.54mm_Vertical
- removed JP4: 2-10, Connector_PinHeader_2.54mm:PinHeader_1x02_P2.54mm_Vertical
- removed the REF** at (-9.00, 79.0)
- added Q1: 2N7000, Package_TO_SOT_THT:TO-92_Inline, F.Cu at (-17.1, 55.2)
- added Q2: 2N7000, Package_TO_SOT_THT:TO-92_Inline, F.Cu at (-11.4, 55.2)
- added Q3: 2N7000, Package_TO_SOT_THT:TO-92_Inline, F.Cu at (-5.71, 55.2)
- added Q4: 2N7000, Package_TO_SOT_THT:TO-92_Inline, F.Cu at (0.00, 55.2)
- added Q5: 2N7000, Package_TO_SOT_THT:TO-92_Inline, F.Cu at (5.71, 55.2)
- added R1: 10K, Resistor_THT:R_Axial_DIN0207_L6.3mm_D2.5mm_P2.54mm_Vertical, F.Cu at (-17.1, 59.1)
- added R10: 10K, Resistor_THT:R_Axial_DIN0207_L6.3mm_D2.5mm_P2.54mm_Vertical, F.Cu at (-3.17, 61.6)
- added R11: 10K, Resistor_THT:R_Axial_DIN0207_L6.3mm_D2.5mm_P2.54mm_Vertical, F.Cu at (0.00, 59.1)
- added R12: 10K, Resistor_THT:R_Axial_DIN0207_L6.3mm_D2.5mm_P2.54mm_Vertical, F.Cu at (2.54, 61.6)
- added R13: 10K, Resistor_THT:R_Axial_DIN0207_L6.3mm_D2.5mm_P2.54mm_Vertical, F.Cu at (5.71, 59.1)
- added R14: 10K, Resistor_THT:R_Axial_DIN0207_L6.3mm_D2.5mm_P2.54mm_Vertical, F.Cu at (8.26, 61.6)
- added R18: 4K7, Resistor_THT:R_Axial_DIN0204_L3.6mm_D1.6mm_P5.08mm_Horizontal, F.Cu at (19.1, 37.5)
- added R2: 10K, Resistor_THT:R_Axial_DIN0207_L6.3mm_D2.5mm_P2.54mm_Vertical, F.Cu at (-14.6, 61.6)
- added R7: 10K, Resistor_THT:R_Axial_DIN0207_L6.3mm_D2.5mm_P2.54mm_Vertical, F.Cu at (-11.4, 59.1)
- added R9: 10K, Resistor_THT:R_Axial_DIN0207_L6.3mm_D2.5mm_P2.54mm_Vertical, F.Cu at (-5.71, 59.1)
- R8: value 4K7 -> 10K; footprint Resistor_THT:R_Axial_DIN0204_L3.6mm_D1.6mm_P5.08mm_Horizontal -> Resistor_THT:R_Axial_DIN0207_L6.3mm_D2.5mm_P2.54mm_Vertical
- SW1: value PRGW0 -> PRG0; footprint Button_Switch_THT:KSA_Tactile_SPST -> Button_Switch_THT:SW_TH_Tactile_Omron_B3F-10xx
- SW2: value PRGW1 -> PRG1; footprint Button_Switch_THT:KSA_Tactile_SPST -> Button_Switch_THT:SW_TH_Tactile_Omron_B3F-10xx
- moved R8 37.8 mm to (-8.89, 61.6), turned to 90 degrees
- moved C1 26.9 mm to (36.8, 73.0)
- moved R6 16.6 mm to (-5.71, 68.6), turned to 270 degrees
- moved U3 16.3 mm to (-9.53, 86.4), turned to 180 degrees
- moved R5 11.4 mm to (-5.71, 73.7), turned to 270 degrees
- moved R3 7.75 mm to (-5.71, 83.8), turned to 270 degrees
- moved R4 7.73 mm to (-5.71, 78.7), turned to 270 degrees
- moved JP5 6.84 mm to (21.6, 29.2), turned to 90 degrees
- moved SW1 4.84 mm to (25.4, 40.6), turned to 0 degrees
- moved SW2 4.45 mm to (35.1, 40.6), turned to 0 degrees
- moved D1 2.62 mm to (8.89, 78.1)
- moved R20 1.27 mm to (19.1, 32.4)
- moved R19 1.27 mm to (24.1, 34.9)
- moved U1 1.27 mm to (-15.9, 41.9)
- moved U2 1.27 mm to (-10.2, 41.9)
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- renumbered R5 to R15, R6 to R16, R7 to R17, R9 to R19, R10 to R20, R1 to R3, R2 to R4, R3 to R5, R4 to R6
Connections:
- R4 pad 1: Net-(J1-Pad2) -> Net-(R4-Pad1)
- R4 pad 2: Net-(R2-Pad2) -> Net-(J1-Pad2)
- R6 pad 1: Net-(J1-Pad4) -> Net-(R6-Pad1)
- R6 pad 2: Net-(R4-Pad2) -> Net-(J1-Pad4)
- R8 pad 1: GND -> Net-(C1-Pad1)
- R8 pad 2: Net-(R8-Pad2) -> Net-(Q2-Pad3)
- SW1 pad 2: Net-(SW1-Pad2) -> (no net)
- SW1 pad 3: (no net) -> Net-(SW1-Pad3)
- SW2 pad 1: Net-(SW2-Pad1) -> GND
- SW2 pad 2: GND -> (no net)
- SW2 pad 3: (no net) -> Net-(SW2-Pad3)
- U1 pad 3: Net-(U1-Pad3) -> Net-(Q1-Pad3)
- U1 pad 7: Net-(J2-Pad2) -> Net-(J2-Pad6)
- U2 pad 1: Net-(J2-Pad3) -> Net-(J2-Pad2)
- U2 pad 3: Net-(U2-Pad3) -> Net-(Q2-Pad3)
- U2 pad 7: Net-(J2-Pad4) -> Net-(J2-Pad7)
- U3 pad 4: Net-(R2-Pad2) -> Net-(R4-Pad1)
- U3 pad 8: Net-(R4-Pad2) -> Net-(R6-Pad1)
- U4 pad 1: Net-(J2-Pad5) -> Net-(J2-Pad3)
- U4 pad 3: Net-(U4-Pad3) -> Net-(Q3-Pad3)
- U4 pad 7: Net-(J2-Pad6) -> Net-(J2-Pad8)
- U5 pad 1: Net-(J2-Pad7) -> Net-(J2-Pad4)
- U5 pad 3: Net-(U5-Pad3) -> Net-(Q4-Pad3)
- U5 pad 7: Net-(J2-Pad8) -> Net-(J2-Pad9)
- U6 pad 1: Net-(J2-Pad9) -> Net-(J2-Pad5)
- U6 pad 3: Net-(U6-Pad3) -> Net-(Q5-Pad3)
- U7 pad 16: Net-(U3-Pad15) -> Net-(Q1-Pad1)
- U7 pad 17: Net-(U3-Pad14) -> Net-(Q2-Pad1)
- U7 pad 18: Net-(U3-Pad11) -> Net-(Q3-Pad1)
- U7 pad 19: Net-(U3-Pad10) -> Net-(Q4-Pad1)
- U7 pad 2: Net-(SW2-Pad1) -> Net-(SW2-Pad3)
- U7 pad 20: Net-(U6-Pad3) -> Net-(Q5-Pad1)
- U7 pad 21: Net-(U5-Pad3) -> Net-(U3-Pad10)
- U7 pad 22: Net-(U4-Pad3) -> Net-(U3-Pad11)
- U7 pad 23: Net-(U2-Pad3) -> Net-(U3-Pad14)
- U7 pad 24: Net-(U1-Pad3) -> Net-(U3-Pad15)
- U7 pad 25: Net-(SW1-Pad2) -> Net-(SW1-Pad3)
- U7 pad 26: (no net) -> Net-(Q1-Pad2)
- U9 pad 8: Net-(R8-Pad2) -> Net-(R18-Pad2)
Routing:
- net Net-(Q1-Pad2): track 0.00 -> 91.4 mm
- net Net-(U1-Pad3): track 64.1 -> 0.00 mm
- net Net-(J2-Pad2): track 73.3 -> 18.2 mm
- net Net-(U2-Pad3): track 53.8 -> 0.00 mm
- net Net-(U4-Pad3): track 46.7 -> 0.00 mm
- net Net-(SW2-Pad3): track 0.00 -> 45.9 mm
- net Net-(SW2-Pad1): track 45.7 -> 0.00 mm
- net Net-(SW1-Pad2): track 42.1 -> 0.00 mm
- net Net-(C1-Pad1): track 118.6 -> 160.5 mm
- net Net-(U5-Pad3): track 41.4 -> 0.00 mm
- net Net-(Q1-Pad1): track 0.00 -> 40.9 mm
- net Net-(SW1-Pad3): track 0.00 -> 38.6 mm
- net Net-(Q2-Pad1): track 0.00 -> 36.6 mm
- net Net-(Q3-Pad1): track 0.00 -> 32.5 mm
- net Net-(U6-Pad3): track 32.0 -> 0.00 mm
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
Commit message: Revised PCB
Parts:
- added REF**: MountingHole_2.7mm_M2.5, MountingHole:MountingHole_2.7mm_M2.5, F.Cu at (-9.00, 79.0)
- moved U3 17.0 mm to (-17.1, 71.1), turned to 90 degrees
- moved R3 13.5 mm to (-15.2, 74.3), turned to 180 degrees
- moved R6 9.03 mm to (1.27, 74.3), turned to 180 degrees
- moved R4 7.75 mm to (-12.1, 74.3), turned to 0 degrees
- moved R1 1.91 mm to (-17.1, 57.1)
- moved R10 1.91 mm to (-3.17, 59.7)
- moved R11 1.91 mm to (0.00, 57.1)
- moved R12 1.91 mm to (2.54, 59.7)
- moved R13 1.91 mm to (5.71, 57.1)
- moved R14 1.91 mm to (8.26, 59.7)
- moved R2 1.91 mm to (-14.6, 59.7)
- moved R7 1.91 mm to (-11.4, 57.1)
- moved R8 1.91 mm to (-8.89, 59.7)
- moved R9 1.91 mm to (-5.71, 57.1)
- moved Q1 1.90 mm to (-17.1, 53.3)
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Connections:
- R4 pad 1: Net-(R4-Pad1) -> Net-(J1-Pad2)
- R4 pad 2: Net-(J1-Pad2) -> Net-(R4-Pad2)
- U1 pad 7: Net-(J2-Pad6) -> Net-(J2-Pad2)
- U2 pad 1: Net-(J2-Pad2) -> Net-(J2-Pad3)
- U2 pad 7: Net-(J2-Pad7) -> Net-(J2-Pad4)
- U3 pad 4: Net-(R4-Pad1) -> Net-(R4-Pad2)
- U4 pad 1: Net-(J2-Pad3) -> Net-(J2-Pad5)
- U4 pad 7: Net-(J2-Pad8) -> Net-(J2-Pad6)
- U5 pad 1: Net-(J2-Pad4) -> Net-(J2-Pad7)
- U5 pad 7: Net-(J2-Pad9) -> Net-(J2-Pad8)
- U6 pad 1: Net-(J2-Pad5) -> Net-(J2-Pad9)
- U7 pad 27: (no net) -> GND
Routing:
- net Net-(J2-Pad7): track 46.3 -> 17.4 mm
- net Net-(Q1-Pad2): track 91.4 -> 116.6 mm
- net Net-(C1-Pad1): track 160.5 -> 185.2 mm
- net Net-(J2-Pad9): track 40.0 -> 16.8 mm
- net Net-(J2-Pad4): track 13.5 -> 36.1 mm
- net Net-(U3-Pad10): track 40.0 -> 20.1 mm
- net Net-(U3-Pad11): track 42.2 -> 23.7 mm
- net Net-(D1-Pad2): track 57.7 -> 39.5 mm
- net Net-(J2-Pad2): track 18.2 -> 36.3 mm
- net Net-(J1-Pad1): track 4.71 -> 21.7 mm
- net Net-(U3-Pad14): track 49.4 -> 32.4 mm
- net Net-(J2-Pad6): track 49.5 -> 36.0 mm
- net Net-(U3-Pad15): track 48.9 -> 36.0 mm
- net Net-(J1-Pad2): track 8.52 -> 19.5 mm
- net Net-(J2-Pad8): track 43.2 -> 35.2 mm
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Other:
- board text added: "WINCTL 1.1"
- board text removed: "WINCTL 1.0"
