File: modules/THR100/hardware/1.0/kicad/THR100.sch (KiCad schematic (older format))
At the start: 45 parts, among them J1 CAN, J2 SWITCHES, J3 Screw_Terminal_01x02, J4 Screw_Terminal_01x02, K1 FINDER-32.21-x300, K2 FINDER-32.21-x300, Q1 NTE123A, Q2 NTE123A, SW1 SCR, SW2 MODE, SW3 INSTANCE, U1 MCP2551-I-P, U2 TMR-1-1211, U3 PDJR_Teensy_3.2, U4 CNY74-2H

Commit message: Revised PCB for analog control
Parts:
- removed SW1: SCR, Button_Switch_THT:SW_DIP_SPSTx01_Slide_6.7x4.1mm_W7.62mm_P2.54mm_LowProfile, symbol Switch:SW_DIP_x01
- added SW1: MODEA, Package_DIP:DIP-4_W7.62mm, symbol Switch:SW_DIP_x02
- SW2: value MODE -> MODEB
- U3: symbol Teensy:PDJR_Teensy_3.2 -> THR100-rescue:PDJR_Teensy_3.2-Teensy
- U4: symbol Teensy:PDJR_CNY74-2H -> THR100-rescue:PDJR_CNY74-2H-Teensy
- renumbered D2 to D1, D3 to D2, D4 to D3, D5 to D4, D6 to D5, D7 to D6, D8 to D7, D9 to D8, D10 to D9, R11 to R10, R12 to R11, R13 to R12, R14 to R13, R15 to R14, R5 to R4, R6 to R5, R7 to R6, R8 to R7, R9 to R8, R10 to R9
Connections:
- net CAN_SCR: now also SW1.4
- net GND: now also SW1.1; no longer SW2.1, SW2.2, SW3.1, SW3.2, SW3.3, SW3.4, SW3.5, SW3.6, SW3.7, SW3.8
- net ANALOG: now reaches U3.22 (D20)
- net ANALOG: now also SW1.3
- net PS_ADC: now reaches U3.23 (D21)
- net SB_ADC: now reaches U3.24 (D22)
- new net: SW2.2, SW3.1, SW3.2, SW3.3, SW3.4, SW3.5, SW3.6, SW3.7, SW3.8
- new net: SW1.2, SW2.1
- no-connect marks 9 -> 5
