File: modules/THR100/hardware/1.0/kicad/THR100.sch (KiCad schematic (older format))
At the start: 46 parts, among them J1 SWITCHES, J2 ANALOG_IN, J3 Screw_Terminal_01x02, J4 Screw_Terminal_01x02, J5 CAN, K1 FINDER-32.21-x300, K2 FINDER-32.21-x300, Q1 NTE123A, Q2 NTE123A, SW1 MODEA, SW2 MODEB, SW3 INSTANCE, U1 CNY74-2H, U2 PDJR_Teensy_3.2, U3 TMR-1-1211, U4 MCP2551-I-P

Commit message: PCB tweak
Parts:
- removed U1: CNY74-2H, Package_DIP:DIP-8-16_W7.62mm, symbol THR100-rescue:PDJR_CNY74-2H-Teensy
- removed U2: PDJR_Teensy_3.2, PDJR2:Teensy30_31_32_LC, symbol THR100-rescue:PDJR_Teensy_3.2-Teensy
- added U3: Teensy_3.2, Package_DIP:DIP-28_W15.24mm_Socket, symbol PDJR:Teensy_3.2
- added U4: CNY74-2H, Package_DIP:DIP-8_W7.62mm, symbol PDJR:CNY74-2H
- SW1: value MODEA -> MISC
- SW2: value MODEB -> MODE
- renumbered C4 to C1, C5 to C2, C6 to C3, C1 to C4, C2 to C5, C3 to C6, D6 to D1, D5 to D2, D9 to D3, D1 to D4, D2 to D5, D4 to D6, D8 to D7, D3 to D8, D7 to D9, J5 to J1, J1 to J2, J2 to J3, J3 to J4, J4 to J5, R14 to R1, R8 to R10, R1 to R11, R2 to R12, R6 to R13, R11 to R14, R12 to R2, R13 to R3, R7 to R4, R4 to R5, R9 to R6, R5 to R7, R10 to R8, R3 to R9, U4 to U1, U3 to U2
Connections:
- net +5V: now also U3.28 (VIN)
- net ADDR_0: now also U3.14 (D12)
- net ADDR_1: now also U3.13 (D11)
- net ADDR_2: now also U3.12 (D10/TX2)
- net ADDR_3: now also U3.11 (D9/RX2)
- net ADDR_4: now also U3.10 (D8/TX3)
- net ADDR_5: now also U3.9 (D7/RX3)
- net ADDR_6: now also U3.8 (D6)
- net ADDR_7: now also U3.7 (D5/TX1)
- net ANALOG: now also U3.22 (D20)
- net CAN_RX: now also U3.6 (D4/CANRX)
- net CAN_TX: now also U3.5 (D3/CANTX)
- net COMMON: now also U3.17 (D15)
- net GND: now also U3.1 (GND), U3.27 (AGND), U4.5, U4.8
- net LED_PWR: now also U3.4 (D2)
- net MODE_SEL: now also U3.16 (D14)
- net PS_ADC: now also U3.23 (D21)
- net PS_CMD: now also U3.3 (D1/TX1), U4.6
- net PS_RLY: now also U3.18 (D16)
- net SB_ADC: now also U3.24 (D22)
- net SB_CMD: now also U3.2 (D0/RX1), U4.7
- net SB_RLY: now also U3.19 (D17)
- net at R11.2: now also U4.1
- net at D4.2 (A): now also U4.2
- net at D5.2 (A): now also U4.3
- net at R12.2: now also U4.4
- no-connect marks 5 -> 6
